File: pcbs/SHEGO75-V2.2/SHEGO75-V2.2.kicad_sch (KiCad schematic)
At the start: 78 parts, among them Q1 AO3401A, Q2 AO3401A, Q3 BSS138, U1 AP2112K-3.3, U2 AP2112K-3.3, U3 W25Q128JVS, U4 SN74LV1T125DBV, U5 RP2040, U6 ESP32-PICO-D4, Y1 12MHz

Commit message: Minor adjustments, tidied schematic
Parts:
- added D1: RED, LED_SMD:LED_0603_1608Metric, symbol PCM_LED_AKL:LED_0603
- added R17: 10K, Mars_Library:R_0603, symbol Mars_Library:R_0603
- added R20, R21: 0, Mars_Library:R_0603, symbol Mars_Library:R_0603
- BOOT1, EN1, ENC1, JST1, TFT1, UART1: now left out of the parts list
- C1: renamed from C7; footprint Capacitor_SMD:C_0402_1005Metric_Pad0.74x0.62mm_HandSolder -> Mars_Library:C_0402
- C10: renamed from C16; footprint Capacitor_SMD:C_0402_1005Metric_Pad0.74x0.62mm_HandSolder -> Mars_Library:C_0402
- C11: renamed from C17; footprint Capacitor_SMD:C_0402_1005Metric_Pad0.74x0.62mm_HandSolder -> Mars_Library:C_0402
- C12: renamed from C18; footprint Capacitor_SMD:C_0805_2012Metric -> Mars_Library:C_0805
- C13: renamed from C19; footprint Capacitor_SMD:C_0805_2012Metric -> Mars_Library:C_0805
- C16: renamed from C22; footprint Capacitor_SMD:C_0603_1608Metric_Pad1.08x0.95mm_HandSolder -> Mars_Library:C_0603
- C17: renamed from C23; footprint Capacitor_SMD:C_0603_1608Metric_Pad1.08x0.95mm_HandSolder -> Mars_Library:C_0603
- C18: renamed from C24; footprint Capacitor_SMD:C_0603_1608Metric -> Mars_Library:C_0603
- C19: renamed from C1; footprint Capacitor_SMD:C_1206_3216Metric -> Mars_Library:C_0603
- C2: renamed from C8; footprint Capacitor_SMD:C_0402_1005Metric_Pad0.74x0.62mm_HandSolder -> Mars_Library:C_0402
- C20: renamed from C2; footprint Capacitor_SMD:C_1206_3216Metric -> Mars_Library:C_0603
- C21: renamed from C3; footprint Capacitor_SMD:C_1206_3216Metric -> Mars_Library:C_0603
- C22: renamed from C4; footprint Capacitor_SMD:C_1206_3216Metric -> Mars_Library:C_0805
- C25, C26: footprint Capacitor_SMD:C_0603_1608Metric -> Mars_Library:C_0603; LCSC (none) -> C1658
- C3: renamed from C9; footprint Capacitor_SMD:C_0402_1005Metric_Pad0.74x0.62mm_HandSolder -> Mars_Library:C_0402
- C30: footprint Mars_Library:R_0603 -> Mars_Library:C_0603
- C4: renamed from C10; footprint Capacitor_SMD:C_0402_1005Metric_Pad0.74x0.62mm_HandSolder -> Mars_Library:C_0402
- C5: renamed from C11; footprint Capacitor_SMD:C_0402_1005Metric_Pad0.74x0.62mm_HandSolder -> Mars_Library:C_0402
- C6: renamed from C12; footprint Capacitor_SMD:C_0402_1005Metric_Pad0.74x0.62mm_HandSolder -> Mars_Library:C_0402
- C7: renamed from C13; footprint Capacitor_SMD:C_0402_1005Metric_Pad0.74x0.62mm_HandSolder -> Mars_Library:C_0402
- C8: renamed from C14; footprint Capacitor_SMD:C_0402_1005Metric_Pad0.74x0.62mm_HandSolder -> Mars_Library:C_0402
- C9: renamed from C15; footprint Capacitor_SMD:C_0402_1005Metric_Pad0.74x0.62mm_HandSolder -> Mars_Library:C_0402
- FB1, FB2: footprint PCM_Ferrite_SMD_Handsoldering_AKL:Ferrite_0805_2012Metric_Pad1.05x1.20mm_BigPads -> Mars_Library:Ferrite_0805
- Q3: value BSS138 -> AO3400A; symbol Transistor_FET:BSS138 -> Mars_Transistor:AO3400A; LCSC (none) -> C20917
- R1: renamed from R3; footprint Resistor_SMD:R_0603_1608Metric -> Mars_Library:R_0603
- R15: renamed from R14; footprint Resistor_SMD:R_0603_1608Metric -> Mars_Library:R_0603
- R16: renamed from R15; footprint Resistor_SMD:R_0603_1608Metric -> Mars_Library:R_0603
- R2: renamed from R4; footprint Resistor_SMD:R_0603_1608Metric -> Mars_Library:R_0603
- R3: renamed from R1; footprint Resistor_SMD:R_0603_1608Metric_Pad0.98x0.95mm_HandSolder -> Mars_Library:R_0603
- R4: renamed from R2; footprint Resistor_SMD:R_0603_1608Metric_Pad0.98x0.95mm_HandSolder -> Mars_Library:R_0603
- R5: value 100R -> 100
- R9: renamed from R7; value 100R -> 100
- SWD1: footprint Mars_Library:Circle_PinHeader_1x04_P2.54mm_4P -> Mars_Library:SWD_Debug_PinHeader_1x04_P2.54mm; now left out of the parts list
- SWD2: footprint Mars_Library:Circle_PinHeader_1x04_P2.54mm_4P -> Mars_Library:SWD_Debug_PinHeader_1x04_P2.54mm; Specifications HEADER 1x4 MALE PINS 0.100” 180deg -> HEADER 1x4 MALE PINS 2.54mm” 180deg; now left out of the parts list
- U6: footprint Package_DFN_QFN:QFN-48-1EP_7x7mm_P0.5mm_EP5.3x5.3mm -> Mars_Library:QFN-48-1EP_7x7mm_P0.5mm_EP5.3x5.3mm_ExtendedPads
- Y1: LCSC (none) -> C9002
- renumbered C20 to C14, C21 to C15, C5 to C23, C6 to C24, R11 to R10, R9 to R11, R18 to R12, R12 to R13, R13 to R14, R16 to R18, R17 to R19, R8 to R7, R10 to R8, U4 to U3, U3 to U4
Connections:
- net GND: now also D1.1 (K)
- net at U6.10 (IO34): now also R17.1
- net IO14_ESP_SCL: now reaches U6.17 (IO14)
- net IO14_ESP_SCL: now also R21.1
- net IO13_ESP_SDA: now reaches U6.20 (IO13)
- net IO13_ESP_SDA: now also R20.1
- net GP20 renamed GP20_SDA
- net GP20_SDA: now also R20.2
- net GP21 renamed GP21_SCL
- net GP21_SCL: now also R21.2
- net GP2_LED_EN renamed GPIO2
- new net: D1.2 (A), R17.2
Other:
- note added: "81 key, 10 ambient, 3 status = 94 LEDs total"
- note added: "ESP32-PICO-D4"
- note added: "Flash + Boot"
- note added: "LED rail decoupling"
- note added: "RP2040"
- note added: "RP2040-to-ESP32 I2C"
- note added: "Small filter"
- note added: "v2.2 connected ESP32 via I2C v2.2 added blink led to ESP32 IO34 v2.2 moved UART connection from GP0+GP1 to GP20+GP21"
- note removed: "81, 10 ambient, 3 status = 94 LEDs total"
- note removed: "ESP32-PICO-D4 + Decoupling"
- note removed: "Flash"
- note removed: "RP2040 + Decoupling"
- moved on the sheet: BOOT1, C1, C10, C11, C12, C13, C14, C15, C16, C17, C18, C19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
