File: pcbs/SHEGO75-V2.2/leds.kicad_sch (KiCad schematic)
At the start: 192 parts, among them J1 LED_EXP

Commit message: Minor adjustments, tidied schematic
Parts:
- AMB1, AMB10, AMB2, AMB3, AMB4, AMB5, AMB6, AMB7, AMB8, AMB9, GLO1, GLO2, GLO3, LED1, LED10, LED11, LED12, LED13, LED14, LED15, LED16, LED17, LED18, LED19, LED2, LED20, LED21, LED22, LED23, LED24, LED25, LED26, LED27, LED28, LED29, LED3, LED30, LED31, LED32, LED33, LED34, LED35, LED36, LED37, LED38, LED39, LED4, LED40, LED41, LED42, LED43, LED44, LED45, LED46, LED47, LED48, LED49, LED5, LED50, LED51, LED52, LED53, LED54, LED55, LED56, LED57, LED58, LED59, LED6, LED60, LED61, LED62, LED63, LED64, LED65, LED66, LED67, LED68, LED69, LED7, LED70, LED71, LED72, LED73, LED74, LED75, LED76, LED77, LED78, LED79, LED8, LED80, LED81, LED9: LCSC (none) -> C5149201
- CA1, CA10, CA2, CA3, CA4, CA5, CA6, CA7, CA8, CA9, CG2: footprint Capacitor_SMD:C_0402_1005Metric_Pad0.74x0.62mm_HandSolder -> Mars_Library:C_0402
- CG1: renamed from CG3; footprint Capacitor_SMD:C_0402_1005Metric_Pad0.74x0.62mm_HandSolder -> Mars_Library:C_0402
- CG3: renamed from CG1; footprint Capacitor_SMD:C_0402_1005Metric_Pad0.74x0.62mm_HandSolder -> Mars_Library:C_0402
- CL1, CL10, CL11, CL12, CL13, CL14, CL15, CL16, CL17, CL18, CL19, CL2, CL20, CL21, CL22, CL23, CL24, CL25, CL26, CL27, CL28, CL29, CL3, CL30, CL31, CL32, CL33, CL34, CL35, CL36, CL37, CL38, CL39, CL4, CL40, CL41, CL42, CL43, CL44, CL45, CL46, CL47, CL48, CL49, CL5, CL50, CL51, CL52, CL53, CL54, CL55, CL56, CL57, CL58, CL59, CL6, CL60, CL61, CL62, CL63, CL64, CL65, CL66, CL67, CL68, CL69, CL7, CL70, CL71, CL72, CL73, CL74, CL75, CL76, CL77, CL78, CL79, CL8, CL80, CL81, CL9: footprint Capacitor_SMD:C_0603_1608Metric_Pad1.08x0.95mm_HandSolder -> Mars_Library:C_0603
- J1: now left out of the parts list
- R22: renamed from R19; footprint Resistor_SMD:R_0603_1608Metric -> Mars_Library:R_0603
- R23: renamed from R20; footprint Resistor_SMD:R_0603_1608Metric_Pad0.98x0.95mm_HandSolder -> Mars_Library:R_0603
- R24: renamed from R21; footprint Resistor_SMD:R_0603_1608Metric_Pad0.98x0.95mm_HandSolder -> Mars_Library:R_0603
Other:
- note added: "Ambient"
- note added: "Expansion"
- note added: "Main"
- note added: "Status"
- moved on the sheet: AMB1, AMB10, AMB2, AMB3, AMB4, AMB5, AMB6, AMB7, AMB8, AMB9, CA1, CA10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
