File: pcbs/SHEGO75-V2.2/sensors.kicad_sch (KiCad schematic)
At the start: 87 parts

Commit message: Minor adjustments, tidied schematic
Parts:
- HE1: value Esc -> 49E; LCSC (none) -> C7420984
- HE10: value F9 -> 49E; LCSC (none) -> C7420984
- HE11: value F10 -> 49E; LCSC (none) -> C7420984
- HE12: value F11 -> 49E; LCSC (none) -> C7420984
- HE13: value F12 -> 49E; LCSC (none) -> C7420984
- HE14: value Del -> 49E; LCSC (none) -> C7420984
- HE15: value `¬ -> 49E; LCSC (none) -> C7420984
- HE16: value 1 -> 49E; LCSC (none) -> C7420984
- HE17: value 2 -> 49E; LCSC (none) -> C7420984
- HE18: value 3 -> 49E; LCSC (none) -> C7420984
- HE19: value 4 -> 49E; LCSC (none) -> C7420984
- HE2: value F1 -> 49E; LCSC (none) -> C7420984
- HE20: value 5 -> 49E; LCSC (none) -> C7420984
- HE21: value 6 -> 49E; LCSC (none) -> C7420984
- HE22: value 7 -> 49E; LCSC (none) -> C7420984
- HE23: value 8 -> 49E; LCSC (none) -> C7420984
- HE24: value 9 -> 49E; LCSC (none) -> C7420984
- HE25: value 0 -> 49E; LCSC (none) -> C7420984
- HE26: value - -> 49E; LCSC (none) -> C7420984
- HE27: value = -> 49E; LCSC (none) -> C7420984
- HE28: value Back -> 49E; LCSC (none) -> C7420984
- HE29: value Home -> 49E; LCSC (none) -> C7420984
- HE3: value F2 -> 49E; LCSC (none) -> C7420984
- HE30: value Tab -> 49E; LCSC (none) -> C7420984
- HE31: value Q -> 49E; LCSC (none) -> C7420984
- HE32: value W -> 49E; LCSC (none) -> C7420984
- HE33: value E -> 49E; LCSC (none) -> C7420984
- HE34: value R -> 49E; LCSC (none) -> C7420984
- HE35: value T -> 49E; LCSC (none) -> C7420984
- HE36: value Y -> 49E; LCSC (none) -> C7420984
- HE37: value U -> 49E; LCSC (none) -> C7420984
- HE38: value I -> 49E; LCSC (none) -> C7420984
- HE39: value O -> 49E; LCSC (none) -> C7420984
- HE4: value F3 -> 49E; LCSC (none) -> C7420984
- HE40: value P -> 49E; LCSC (none) -> C7420984
- HE41: value [ -> 49E; LCSC (none) -> C7420984
- HE42: value ] -> 49E; LCSC (none) -> C7420984
- HE43: value \ -> 49E; LCSC (none) -> C7420984
- HE44: value PgUp -> 49E; LCSC (none) -> C7420984
- HE45: value Caps -> 49E; LCSC (none) -> C7420984
- HE46: value A -> 49E; LCSC (none) -> C7420984
- HE47: value S -> 49E; LCSC (none) -> C7420984
- HE48: value D -> 49E; LCSC (none) -> C7420984
- HE49: value F -> 49E; LCSC (none) -> C7420984
- HE5: value F4 -> 49E; LCSC (none) -> C7420984
- HE50: value G -> 49E; LCSC (none) -> C7420984
- HE51: value H -> 49E; LCSC (none) -> C7420984
- HE52: value J -> 49E; LCSC (none) -> C7420984
- HE53: value K -> 49E; LCSC (none) -> C7420984
- HE54: value L -> 49E; LCSC (none) -> C7420984
- HE55: value ; -> 49E; LCSC (none) -> C7420984
- HE56: value ' -> 49E; LCSC (none) -> C7420984
- HE57: value Enter -> 49E; LCSC (none) -> C7420984
- HE58: value PgDn -> 49E; LCSC (none) -> C7420984
- HE59: value L_Shift -> 49E; LCSC (none) -> C7420984
- HE6: value F5 -> 49E; LCSC (none) -> C7420984
- HE60: value Z -> 49E; LCSC (none) -> C7420984
- HE61: value X -> 49E; LCSC (none) -> C7420984
- HE62: value C -> 49E; LCSC (none) -> C7420984
- HE63: value V -> 49E; LCSC (none) -> C7420984
- HE64: value B -> 49E; LCSC (none) -> C7420984
- HE65: value N -> 49E; LCSC (none) -> C7420984
- HE66: value M -> 49E; LCSC (none) -> C7420984
- HE67: value , -> 49E; LCSC (none) -> C7420984
- HE68: value . -> 49E; LCSC (none) -> C7420984
- HE69: value / -> 49E; LCSC (none) -> C7420984
- HE7: value F6 -> 49E; LCSC (none) -> C7420984
- HE70: value R_Shift -> 49E; LCSC (none) -> C7420984
- HE71: value Up -> 49E; LCSC (none) -> C7420984
- HE72: value L_Ctrl -> 49E; LCSC (none) -> C7420984
- HE73: value Code -> 49E; LCSC (none) -> C7420984
- HE74: value L_alt -> 49E; LCSC (none) -> C7420984
- HE75: value Space -> 49E; LCSC (none) -> C7420984
- HE76: value R_Alt -> 49E; LCSC (none) -> C7420984
- HE77: value Fn -> 49E; LCSC (none) -> C7420984
- HE78: value R_Ctrl -> 49E; LCSC (none) -> C7420984
- HE79: value Left -> 49E; LCSC (none) -> C7420984
- HE8: value F7 -> 49E; LCSC (none) -> C7420984
- HE80: value Down -> 49E; LCSC (none) -> C7420984
- HE81: value Right -> 49E; LCSC (none) -> C7420984
- HE9: value F8 -> 49E; LCSC (none) -> C7420984
- MC1, MC2, MC3: footprint Capacitor_SMD:C_0402_1005Metric_Pad0.74x0.62mm_HandSolder -> Mars_Library:C_0402
- MUX1, MUX2, MUX3: footprint ADG732BSUZ:QFP50P900X900X120-49N -> Package_QFP:TQFP-48_7x7mm_P0.5mm; LCSC (none) -> C114845
Other:
- note added: "KNOB"
- note added: "ST7735 DISPLAY"
- moved on the sheet: HE1, HE10, HE11, HE12, HE13, HE14, HE15, HE16, HE17, HE18, HE19, HE2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
